Commit message: mimic joints > gripper

File: mecanum_description/urdf/mecanum.xacro (robot description, xacro)
@@ -339,4 +339,5 @@
 <joint name="rfinger_mimic" type="continuous">
   <origin xyz="0.016021 -0.018479 -0.018965" rpy="0 0 0"/>
+  <mimic joint="rgear" multiplier="-1"/>
   <parent link="gear1-r4_1"/>
   <child link="Gripper_finger-r4_2"/>
@@ -345,4 +346,5 @@
 <joint name="lfinger_mimic" type="continuous">
   <origin xyz="0.016111 0.017188 -0.02007" rpy="0 0 0"/>
+  <mimic joint="lgear" multiplier="-1"/>
   <parent link="gear2-r4_1"/>
   <child link="Gripper_finger-r4_1"/>
@@ -357,4 +359,5 @@
 <joint name="lgear" type="continuous">
   <origin xyz="0.031814 0.015753 -0.025566" rpy="0 0 0"/>
+  <mimic joint="rgear" multiplier="-1"/>
   <parent link="Gripper_base-r4_1"/>
   <child link="gear2-r4_1"/>

Commit message: added rviz-joint state publisher gui

File: mecanum_description/urdf/mecanum.xacro (robot description, xacro)
@@ -339,5 +339,5 @@
 <joint name="rfinger_mimic" type="continuous">
   <origin xyz="0.016021 -0.018479 -0.018965" rpy="0 0 0"/>
-  <mimic joint="rgear" multiplier="-1"/>
+  <mimic joint="rgear" multiplier="1"/>
   <parent link="gear1-r4_1"/>
   <child link="Gripper_finger-r4_2"/>
